File: ferntypes.kicad_sch (KiCad schematic)
At the start: 15 parts, among them J3 JST SH, J4 Pico EZmate, SW3 SKQGABE010, U2 XC6206PxxxMR-Regulator_Linear, U3 STM32F072C8Tx

Commit message: project
Connections:
- net COL0: now also U3.17 (PA7); no longer U3.16 (PA6)
- net COL1: now also U3.18 (PB0); no longer U3.17 (PA7)
- net COL2: now also U3.19 (PB1); no longer U3.18 (PB0)
- net COL3: now also U3.20 (PB2); no longer U3.19 (PB1)
- net COL4: now also U3.21 (PB10); no longer U3.20 (PB2)
- net COL5: now also U3.22 (PB11); no longer U3.21 (PB10)
- net ROW0: now also U3.16 (PA6); no longer U3.15 (PA5)
- net ROW3: now also U3.15 (PA5); no longer U3.14 (PA4)
- no-connect marks 0 -> 14
Other:
- note added: "DB connectors"
- note added: "boot, etc."
- note added: "decoupling caps"
- note added: "power shifter"
- moved on the sheet: C1, C2, C3, C4, C5, C6, C7, C8, C9, J3, J4, R1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
